Commit message: Add display functions, Fix ant mesh

File: urdf/environment_3d.urdf (robot description, URDF)
Before this commit: robot environment, 11 links, 10 joints
Links:
- removed link l_nine
Joints:
- removed joint j_nine
- joint j_eight: origin xyz=-4 -4 0 rpy=-0.5 -0.5 0 -> xyz=-4.8 -4.8 0 rpy=-0.5 -0.5 -0.5
- joint j_five: origin xyz=4 4 0 rpy=0 -0.4 0 -> xyz=4.7 4 0 rpy=0 -0.4 0
- joint j_four: origin xyz=0 -4 0 rpy=0 -0.1 0 -> xyz=0 -4.7 0 rpy=-0.2 -0.1 0
- joint j_fourfive: origin xyz=0 4 0 rpy=0 0 0 -> xyz=0 4 0 rpy=-0.2 0.1 0
- joint j_one: origin xyz=0 0 0 rpy=0 0 0 -> xyz=0 0 0 rpy=0 -0.1 0
- joint j_seven: origin xyz=-4 4 0 rpy=0.6 -0.3 0 -> xyz=-4 4.7 0 rpy=0.6 -0.3 0.5
- joint j_two: origin xyz=-4 0 0 rpy=0 -0.2 0 -> xyz=-4 0 0 rpy=0.1 -0.2 0

File: urdf/sphere.urdf (robot description, URDF)
Before this commit: robot object, 1 links, 0 joints
Links:
- link base_link: geometry collision sphere radius=0.2; visual sphere radius=0.2
