Commit message: New environment and scripts modifications:
* Add new environment and script for scene_jump
* Add new cone mesh to display friction cones with correct orientation
* Adapt scripts to changes in hpp-corbaserver function (setOrientation, projectOnObstacle)
* New function to display in viewer a path with a chosen number of points

File: urdf/ant_sphere.urdf (robot description, URDF)
Before this commit: robot object, 2 links, 1 joints
Links:
- link base_link: geometry collision sphere radius=0.11; visual mesh filename=package://animals_description/meshes/ant_black.dae
- link l_bounding_sphere: geometry visual sphere radius=0.11
Joints:
- joint j_bounding_sphere: origin xyz=0 0.009 0.03 -> xyz=0 0 0

File: urdf/environment_3d_with_window.urdf (robot description, URDF)
Before this commit: robot environment, 14 links, 13 joints
Links:
- link l_fourteen: geometry collision box size=0.15 2 3; visual box size=0.15 2 3
- link l_twelve: geometry collision box size=0.15 2 3; visual box size=0.15 2 3

File: urdf/scene_jump.urdf (robot description, URDF)
Before this commit: robot object, 1 links, 0 joints
Links:
- link base_link: geometry collision mesh filename=package://animals_description/meshes/scene_jump.dae; visual mesh filename=package://animals_description/meshes/scene_jump.dae

File: urdf/scene_jump_harder.urdf (robot description, URDF)
Before this commit: robot object, 1 links, 0 joints
Links:
- link base_link: geometry collision mesh filename=package://animals_description/meshes/scene_jump5.dae; visual mesh filename=package://animals_description/meshes/scene_jump5.dae
