Commit message: Modifications for cones, environments, scripts:
* scene_jump environment updated to avoid shortcut-jumps
* cave environment updated to remove big unused part (no contact-shoot in it)
* new urdf and mesh for two frictions cones (mu = 0.5 and 1.2)
* remove deprecated meshes
* udpate rabbit and ant with blender-material-color instead of texture
* update scripts to new cones
* add script for rabbit in scene_jump (special theta orientations are given)

File: urdf/ant.urdf (robot description, URDF)
Before this commit: robot object, 1 links, 0 joints
Links:
- link base_link: geometry collision mesh filename=package://animals_description/meshes/ant_black2.dae; visual mesh filename=package://animals_description/meshes/ant_black2.dae

File: urdf/ant_sphere.urdf (robot description, URDF)
Before this commit: robot object, 2 links, 1 joints
Links:
- link base_link: geometry collision sphere radius=0.11; visual mesh filename=package://animals_description/meshes/ant_black2.dae
- link l_bounding_sphere: geometry visual sphere radius=0.13

File: urdf/cave.urdf (robot description, URDF)
Before this commit: robot decor, 1 links, 0 joints
Links:
- link decor_base: geometry collision mesh filename=package://animals_description/meshes/cave_mono2_2.dae; visual mesh filename=package://animals_description/meshes/cave_mono2_2.dae

File: urdf/rabbit.urdf (robot description, URDF)
Before this commit: robot object, 1 links, 0 joints
Links:
- link base_link: geometry collision mesh filename=package://animals_description/meshes/rabbit3.dae; visual mesh filename=package://animals_description/meshes/rabbit3.dae

File: urdf/scene_jump_harder.urdf (robot description, URDF)
Before this commit: robot object, 1 links, 0 joints
Links:
- link base_link: geometry collision mesh filename=package://animals_description/meshes/scene_jump8_2.dae; visual mesh filename=package://animals_description/meshes/scene_jump8_2.dae
