Commit message: Clean package:
* fix doc in robot Python classes
* add lighter colors in box environments (plane...)
* add new meshes for cave (stl)
* add more simple scripts (cave_mono, plane...) to lighten ant / sphere scripts

File: urdf/cave.urdf (robot description, URDF)
Before this commit: robot decor, 1 links, 0 joints
Links:
- link decor_base: geometry collision mesh filename=package://animals_description/meshes/cave_mono3_3.stl; visual mesh filename=package://animals_description/meshes/cave_mono3_3.stl

File: urdf/sphere.urdf (robot description, URDF)
Before this commit: robot object, 1 links, 0 joints
Links:
- link base_link: geometry collision sphere radius=0.02; visual sphere radius=0.02

Commit message: Modify scripts and meshes:
* improve cave mesh, add cylinder object
* add benchmark and run scripts
* improve scene_jump mesh: transparency, smoother polygons
* fix doxygen

File: urdf/cave.urdf (robot description, URDF)
Before this commit: robot decor, 1 links, 0 joints
Links:
- added link l_decor_one; visual mesh filename=package://animals_description/meshes/cave_mono3_3_cylinder_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
- link decor_base: geometry collision mesh filename=package://animals_description/meshes/cave_mono3_3.stl; visual mesh filename=package://animals_description/meshes/cave_mono3_3.dae
Joints:
- added joint j_decor_one: type fixed, parent decor_base, child l_decor_one, origin xyz=0 0 0 rpy=0 0 0

File: urdf/scene_jump_harder.urdf (robot description, URDF)
Before this commit: robot object, 1 links, 0 joints
Links:
- link base_link: geometry collision mesh filename=package://animals_description/meshes/scene_jump10.stl; visual mesh filename=package://animals_description/meshes/scene_jump10.dae

Commit message: Add envir3d_mesh and Blender parts in scripts:
* also add parabResults data in scripts (e.g. "runs")

File: urdf/cave.urdf (robot description, URDF)
Before this commit: robot decor, 2 links, 1 joints
Links:
- removed link l_decor_one
- link decor_base: geometry collision mesh filename=package://animals_description/meshes/cave_mono_short_1.stl; visual mesh filename=package://animals_description/meshes/cave_mono_short_1.dae
Joints:
- removed joint j_decor_one
